Commit message: removed conflicts with jetleg package xacro files

File: urdf/primitives/colors.xacro (robot description, xacro)
@@ -1,18 +1,6 @@
 <?xml version="1.0"?>
 <robot xmlns:xacro="http://www.ros.org/wiki/xacro" name="colors">
-   <material name="white">
+   <material name="white_opaque">
         <color rgba="1 1 1 1"/>
     </material>
-    <material name="red">
-        <color rgba="1 0 0 1"/>
-    </material>
-    <material name="red_transluscent">
-        <color rgba="1 0 0 0.25"/>
-    </material>
-    <material name="white_transluscent">
-        <color rgba="1 1 1 0.25"/>
-    </material>
-    <material name="grey">
-        <color rgba="0.5 0.5 0.5 1"/>
-    </material>
 </robot>

File: urdf/primitives/ramp.xacro (robot description, xacro)
@@ -9,5 +9,5 @@
                     <box size="${length} ${width} ${thickness}"/>
                 </geometry>
-                <material name="white"/>
+                <material name="white_opaque"/>
             </visual>
             <collision>

File: urdf/primitives/staircase.xacro (robot description, xacro)
@@ -7,5 +7,5 @@
                     <box size="${depth} ${width} ${height if height >= 0 else -height}"/>
                 </geometry>
-                <material name="white"/>
+                <material name="white_opaque"/>
             </visual>
             <collision>
