Commit message: create standalone staircase model to load into pybullet simulation

File: urdf/prebuilts/staircase_var1.xacro (robot description, xacro)
@@ -4,4 +4,6 @@
     <xacro:include filename="$(find obstacles)/urdf/primitives/staircase.xacro"/>
     <!-- base_link is not included in this file because it is meant to be integrated with other robots -->
+    <link name="base_link">
+    </link>
     <xacro:macro name="staircase_var1" params="postfix offset_x offset_z">
         <xacro:property name="seg1_quantity" value="10"/>

Commit message: remove base_link from staircase template

File: urdf/prebuilts/staircase_var1.xacro (robot description, xacro)
@@ -4,6 +4,4 @@
     <xacro:include filename="$(find obstacles)/urdf/primitives/staircase.xacro"/>
     <!-- base_link is not included in this file because it is meant to be integrated with other robots -->
-    <link name="base_link">
-    </link>
     <xacro:macro name="staircase_var1" params="postfix offset_x offset_z">
         <xacro:property name="seg1_quantity" value="10"/>
